Commit message: my first commit

File: 8track.urdf (robot description, URDF)
Before this commit: robot robotURDF, 23 links, 26 joints
Links:
- link 8track: geometry collision mesh filename=package://robotURDF/DAEmeshes/spindle.dae scale=1 1 1; visual mesh filename=package://robotURDF/DAEmeshes/8track.dae scale=1 1 1
- link gps_link: geometry collision cylinder length=0.1 radius=0.1; visual cylinder length=0.1 radius=0.1
- link imu_link: geometry collision cylinder length=0.08 radius=0.01; visual cylinder length=0.08 radius=0.01
Joints:
- joint 8joint: origin xyz=0 0 -0.06 rpy=0 -0 0 -> xyz=0 0 -0.1 rpy=0 -0 0
- joint camerachassis_joint: origin xyz=0.25 0 0.12 rpy=0 -0 0 -> xyz=1 0 0 rpy=0 -0 0
